File: hardware/pjc-kicad/pjc-kicad.sch (KiCad schematic (older format))
At the start: 19 parts

Commit message: More work on schematic and moved some stuff around.
Parts:
- removed C?: 100nF, symbol C
- removed R?: 330, symbol R
- added C? (x2): 100nF, symbol C
- added C?: 10uF, symbol CP1
- added CON?: USB-MINI-B, symbol USB-MINI-B
- added CON?: CONN_2, symbol CONN_2
- added CON?: AVR-ISP-10, AVR-ISP-10, symbol AVR-ISP-10
- added CON?: SPRING_TERM_2, symbol SPRING_TERM_2
- added D?: Green, symbol LED
- added D?: Amber, symbol LED
- added D?: Red, symbol LED
- added Q? (x2): MOSFET_P, symbol MOSFET_P
- added R? (x3): 10k, symbol R
- added R? (x3): 470, symbol R
- added U?: FT232RL, symbol FT232RL
- added U?: MCP3302, symbol MCP3302
- gave numbers to parts that had none: 2
Connections:
- net labels added: MISO, MOSI, SCK, UART_RX, UART_TX, USB_VBUS, ~RESET, ~USB_PWREN
- wire segments 66 -> 152
- no-connect marks 0 -> 19
Other:
- moved on the sheet: R?

Commit message: Created thermistor section using MCP3301 ADC and created TMP36 symbol.
Parts:
- removed U?: MCP3302, symbol MCP3302
- added R? (x4): 10k, symbol R
- added U?: MCP3301, symbol MCP3301
Connections:
- net labels added: ~ADC_CS
- wire segments 152 -> 187
Other:
- moved on the sheet: C?, R?, X?

Commit message: Add more datasheets as schematic moves toward completion.
Parts:
- removed F?: 3A Max, symbol FUSE
- added C?: 100nF, symbol C
- added CON? (x4): CONN_2, symbol CONN_2
- added CON?: 4PIN_FAN_CONN, 4PIN_FAN_PTH, symbol 4PIN_FAN_CONN
- added F?: 500mA, symbol VR
- added R?: 10k, symbol R
- added R?: 3.3k, symbol R
- added U?: TMP36_SOIC, SO8E, symbol TMP36_SOIC
- added U? (x4): NUD3124, symbol NUD3124
- added U?: BSP762T, symbol BSP762T
- added U?: SN74LVC1G07, SOT23-5, symbol SN74LVC1G07
Connections:
- net labels added: ANA_12V_FB, ANA_AMBIENT, LAMP_EN, LAMP_PWM, LED_EN_AMBER, LED_EN_GREEN, LED_EN_RED, PROJECTOR_ON, USB_5V
- wire segments 187 -> 253
- no-connect marks 19 -> 20
Other:
- moved on the sheet: C?, CON?, D?, Q?, R?, X?

Commit message: Schematic layout closer to completion
Parts:
- added CON?: CONN_2, symbol CONN_2
- added D?: 4.7V, symbol ZENER
- added R?: 1k, symbol R
Connections:
- wire segments 253 -> 262
Changed lines of the file:
@@
-EESchema Schematic File Version 2  date Sun 13 Jan 2013 11:35:03 PM EST
+EESchema Schematic File Version 2  date Mon 14 Jan 2013 09:36:05 PM EST
 LIBS:power
 LIBS:device
@@
 Sheet 1 1
 Title "Projector Controller Board"
-Date "14 jan 2013"
+Date "15 jan 2013"
 Rev "0"
 Comp ""
@@
 Wire Wire Line
 	13350 12840 13350 12660
+$Comp
+L CONN_2 CON?
+U 1 1 50F4A8EC
+P 10600 2800
+F 0 "CON?" V 10550 2800 40  0000 C CNN
+F 1 "CONN_2" V 10650 2800 40  0000 C CNN
+	1    10600 2800
+	-1   0    0    -1
+$EndComp
+$Comp
+L GND #PWR?
+U 1 1 50F4A8F7
+P 11080 3350
+F 0 "#PWR?" H 11080 3350 30  0001 C CNN
+F 1 "GND" H 11080 3280 30  0001 C CNN
+	1    11080 3350
+	1    0    0    -1
+$EndComp
+Wire Wire Line
+	10950 2900 11080 2900
+Wire Wire Line
+	11080 2900 11080 3270
+Wire Wire Line
+	11080 3270 11080 3350
+$Comp
+L R R?
+U 1 1 50F4AA2E
+P 11400 2700
+F 0 "R?" V 11500 2810 50  0000 C CNN
+F 1 "1k" V 11500 2600 50  0000 C CNN
+	1    11400 2700
+	0    -1   -1   0
+$EndComp
+Wire Wire Line
+	10950 2700 11150 2700
+$Comp
+L ZENER D?
+U 1 1 50F4BF4A
+P 11810 2990
+F 0 "D?" V 11890 2870 50  0000 C CNN
+F 1 "4.7V" V 11770 2850 40  0000 C CNN
+	1    11810 2990
+	0    -1   -1   0
+$EndComp
+Text Label 12010 2700 0    60   ~ 0
+PROJECTOR_ON
+Wire Wire Line
+	11650 2700 11810 2700
+Wire Wire Line
+	11810 2700 12010 2700
+Wire Wire Line
+	11810 2790 11810 2700
+Connection ~ 11810 2700
+Wire Wire Line
+	11810 3190 11810 3270
+Wire Wire Line
+	11810 3270 11080 3270
+Connection ~ 11080 3270
 $EndSCHEMATC

Commit message: lots more datasheets as schematic moves very close to completion
Parts:
- removed CON?: SPRING_TERM_2, symbol SPRING_TERM_2
- removed CON?: CONN_2, symbol CONN_2
- removed D?: 4.7V, symbol ZENER
- removed F?: 500mA, symbol VR
- removed Q?: IRFZ34N, symbol MOSFET_N
- removed Q?: MOSFET_P, symbol MOSFET_P
- removed R?: 10k, symbol R
- removed S?: TAC_SWITCHPTH, SparkFun-TACTILE-PTH, symbol TAC_SWITCHPTH
- added C?: 100nF, symbol C
- added CON?: CONN_2, symbol CONN_2
- added F? (x5): 120mA, symbol VR
- added K?: CONN_3, symbol CONN_3
- added L?: INDUCTOR_SMALL, symbol INDUCTOR_SMALL
- added Q?: RSQ035N03, symbol RSQ035N03
- added R?: 10k, symbol R
- added S?: TAC_SWITCHSMD, SparkFun-TACTILE_SWITCH_SMD, symbol TAC_SWITCHSMD
- added SW?: SWITCH_INV, symbol SWITCH_INV
- added U?: VOM618A-4T, symbol OPTO-TRANSISTOR4
- C? (x2): value 10uF -> 4.7uF
- C?: value 100nF -> 10nF
- D?: value 1N4001 -> S1M
- R?: value 1k -> 3.3k
- U?: value LM7805 -> L78M05C
Connections:
- net labels added: +5V_USB
- net labels removed: USB_5V
- wire segments 262 -> 277
Other:
- moved on the sheet: C?, CON?, Q?, R?, U?, U?A, U?B

Commit message: Schematic mostly complete and reorganized datasheets
Parts:
- removed C? (x2): 4.7uF, symbol CP1
- removed C?: 100uF, symbol CP1
- removed CON?: M025MM, SparkFun-SCREWTERMINAL-5MM-2, symbol M025MM
- removed CON?: CONN_2, symbol CONN_2
- added C?: 100nF, symbol C
- added C?: 4.7uF, symbol C
- added C?: 10uF, symbol C
- added C?: 1uF, symbol C
- added JP?: M023.5MM, SparkFun-SCREWTERMINAL-3.5MM-2, symbol M023.5MM
- added JP?: JUMPER-2PTH, SparkFun-1X02, symbol JUMPER-2PTH
- added MH? (x4): MNT_HOLE_NPT, symbol MNT_HOLE_NPT
- added TP? (x17): TST, symbol TST
- D?: value Amber -> Yellow
- R?: value 10k -> 3.3k
- R?: value 470 -> 1.5k
- R?: value 470 -> 2.2k
Connections:
- net +12V: now also JP?.2
- net +5V: now also C?.1, JP?.1
- net +5V_USB: no longer SW?.1, U?.VO
- net ANA_12V_FB: now also TP?.1
- net GND: now also C?.2, C?.2, C?.2, C?.2
- net LAMP_EN: now also U?.14 ((PCINT0/CLKO/ICP1)PB0); no longer U?.2 (IN), U?.6 ((PCINT20/XCK/T0)PD4)
- net LED_EN_GREEN: now also U?.5 (G); no longer U?.5 (G)
- net LED_EN_RED: now also U?.5 (G); no longer U?.5 (G)
- net PROJECTOR_ON: now also U?.25 ((PCINT10/ADC2)PC2); no longer U?.4 ((PCINT18/INT0)PD2)
- net UART_RX: now also TP?.1
- net UART_TX: now also TP?.1
- net ~ADC_CS: now also TP?.1
- net at R?.1: now also JP?.2; no longer U?.14 ((PCINT0/CLKO/ICP1)PB0)
- net at D?.2 (K), U?.VI: now also C?.1
- net at Q?.1 (D), Q?.2 (D), Q?.3 (G)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: now also JP?.1
- net at C?.1, L?.2, Q?.S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: now also C?.1
- net at R?.1, R?.2, U?.1 (VREF)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: now also TP?.1
- net LAMP_PWM renamed FAN_PWM
- net LED_EN_AMBER renamed LED_EN_YELLOW
- new net: C?.1, SW?.1, TP?.1, U?.VO
- new net FAN_EN: U?.2 (IN), U?.4 ((PCINT18/INT0)PD2)
- no-connect marks 20 -> 24
Other:
- note added: "Analog Inputs"
- note added: "Fan Control"
- note added: "Main Power Input"
- note added: "Microcontroller"
- note added: "Mounting Holes"
- note added: "Programming and Reset"
- note added: "Projector On Input"
- note added: "Relay and LED Outputs"
- note added: "Temperature Input"
- note added: "USB/UART IO"
- moved on the sheet: C?, CON?, D?, F?, K?, L?, Q?, R?, S?, SW?, U?, U?A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

Commit message: Add pull-downs where needed to outputs and fix test points
Parts:
- added R? (x3): 10k, symbol R
Connections:
- net +5V: now also TP?.1
- net +5V_USB: now also TP?.1
- net ANA_AMBIENT: now also TP?.1
- net FAN_EN: now also TP?.1, R?.1
- net FAN_PWM: now also TP?.1, R?.1
- net GND: now also R?.2, R?.2, R?.2
- net LAMP_EN: now also TP?.1, R?.1
- net LED_EN_GREEN: now also TP?.1
- net LED_EN_RED: now also TP?.1
- net LED_EN_YELLOW: now also TP?.1
- net PROJECTOR_ON: now also TP?.1
- net at C?.1, C?.1, L?.2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: now also TP?.1
Other:
- moved on the sheet: CON?, F?, TP?, U?, U?A, U?B
