File: hardware/pjc-kicad/pjc-kicad.kicad_pcb (KiCad board)
At the start: 2 copper layers, 110.5 x 104.1 mm, 88 parts, among them CON1 USB-MINI-B, CON10 CONN_2, CON2 CONN_3, CON3 CONN_2, CON4 M023.5MM, CON5 4PIN_FAN_CONN, CON6 CONN_2, CON7 CONN_2, CON8 AVR-ISP-10, CON9 CONN_2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

Commit message: Changed NPTHs to be PTHs with no pad since otherwise KiCAD will generate two drill files.
KiCAD generates a separate drill file for NPTHs (non-plated through holes), which OSH Park does not want.  Oh, I've decided to manufacture the boards at OSH Park.  Should probably mention that.
Parts:
- moved C14 1.91 mm to (139.7, 132.1)
- moved U9 1.91 mm to (139.7, 139.7)
Routing:
- net GND: track 271.5 -> 258.3 mm, vias 18 -> 17
- net /ANA_AMBIENT: track 40.6 -> 36.9 mm
- net +5V: track 248.4 -> 249.5 mm
Other:
- board text added: "LEDs"
- board text removed: "LEDs:"

Commit message: Just sent board for manufacture!
The modules in pjc.mod that were derived from the SparkFun library had the reference text on the wrong layer, so those had to be corrected by hand.
Parts:
- added G***: OSHW_LOGO_400mil, OSHW_LOGO_400mil, F.Cu at (139.7, 146.3)
- JP1: footprint SparkFun-1X02 -> PIN_ARRAY_2X1
- moved C14 6.29 mm to (135.3, 136.5), turned to 90 degrees
- moved U9 4.49 mm to (142.9, 136.5), turned to 180 degrees
- moved JP1 1.27 mm to (154.9, 81.3)
Routing:
- net GND: track 258.3 -> 278.9 mm, vias 17 -> 18
- net /ANA_AMBIENT: track 36.9 -> 28.0 mm
- net N-0000033: track 30.3 -> 31.5 mm
Other:
- board text added: "Projector Controller"
- board text added: "Reset"
- board text added: "Rev A"
- board text removed: "Projector Controller Rev A"
